File: Hardware/reader.kicad_pcb (KiCad board)
At the start: 2 copper layers, 21 parts, among them IC1 ATTINY2313-P, P1 RST, P3 UART connector, P4 Lock, P6 CONN_01X08, P7 +12V PWR, Q1 BC817-40, Q2 BD237, U1 LM7805CT

Commit message: * EEPROM copy device HW and FW * administration python scripts for EEPROM reader and RFID reader * Python scripts bundled into standalone apps for both Linux and Win
Parts:
- P3: value UART connector -> UART
Changed lines of the file:
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@@
     (links 39)
     (no_connects 0)
-    (area 97.124999 70.125 126.825 123.015)
+    (area 0 0 0 0)
     (thickness 1.6)
     (drawings 0)
@@
     (mod_text_size 1 1)
     (mod_text_width 0.15)
-    (pad_size 1.6 1.6)
-    (pad_drill 0.8)
+    (pad_size 1.5 1.5)
+    (pad_drill 0.6)
     (pad_to_mask_clearance 0)
     (aux_axis_origin 0 0)
-    (visible_elements FFFFEF7F)
+    (visible_elements FFFFFF7F)
     (pcbplotparams
       (layerselection 0x00030_80000001)
@@
       (outputformat 1)
       (mirror false)
-      (drillshape 0)
+      (drillshape 1)
       (scaleselection 1)
       (outputdirectory ""))
@@
       (effects (font (size 1 1) (thickness 0.15)))
     )
-    (fp_text value 100n (at 3.81 0) (layer F.Fab)
+    (fp_text value 100n (at 0 2.1) (layer F.Fab)
       (effects (font (size 1 1) (thickness 0.15)))
     )
@@
       (effects (font (size 1 1) (thickness 0.15)))
     )
-    (fp_text value 10u (at -3.81 0 180) (layer F.Fab)
+    (fp_text value 10u (at 0 2.1 180) (layer F.Fab)
       (effects (font (size 1 1) (thickness 0.15)))
     )
@@
     (descr "LED 3mm round vertical")
     (tags "LED  3mm round vertical")
-    (fp_text reference D1 (at 1.91 3.06 90) (layer F.SilkS) hide
-      (effects (font (size 1 1) (thickness 0.15)))
-    )
-    (fp_text value LED (at -1.27 0 180) (layer F.Fab)
+    (fp_text reference D1 (at 1.91 3.06 90) (layer F.SilkS)
+      (effects (font (size 1 1) (thickness 0.15)))
+    )
+    (fp_text value LED (at 1.3 -2.9 90) (layer F.Fab)
       (effects (font (size 1 1) (thickness 0.15)))
     )
@@
       (effects (font (size 1 1) (thickness 0.15)))
     )
-    (fp_text value "UART connector" (at 3.81 7.62 270) (layer F.Fab)
+    (fp_text value UART (at 0 -2.75 270) (layer F.Fab)
       (effects (font (size 1 1) (thickness 0.15)))
     )
@@
     (descr "Through hole socket strip")
     (tags "socket strip")
-    (fp_text reference P4 (at 0 -5.1 180) (layer F.SilkS) hide
-      (effects (font (size 1 1) (thickness 0.15)))
-    )
-    (fp_text value Lock (at 2.54 -2.54 180) (layer F.Fab)
+    (fp_text reference P4 (at 0 -5.1 180) (layer F.SilkS)
+      (effects (font (size 1 1) (thickness 0.15)))
+    )
+    (fp_text value Lock (at 0 -3.1 180) (layer F.Fab)
       (effects (font (size 1 1) (thickness 0.15)))
     )
@@
     (tags SOT-23)
     (attr smd)
-    (fp_text reference Q1 (at 0 2.5 270) (layer B.SilkS) hide
+    (fp_text reference Q1 (at 0 2.5 270) (layer B.SilkS)
       (effects (font (size 1 1) (thickness 0.15)) (justify mirror))
     )
-    (fp_text value BC817-40 (at 0 6.35 360) (layer B.CrtYd)
+    (fp_text value BC817-40 (at 0 -2.5 270) (layer B.Fab)
       (effects (font (size 1 1) (thickness 0.15)) (justify mirror))
     )
@@
     (tags "resistor 0805")
     (attr smd)
-    (fp_text reference R4 (at 0 -2.1) (layer F.SilkS) hide
-      (effects (font (size 1 1) (thickness 0.15)))
-    )
-    (fp_text value 1K (at -1.27 -1.27) (layer F.Fab)
+    (fp_text reference R4 (at 0 -2.1) (layer F.SilkS)
+      (effects (font (size 1 1) (thickness 0.15)))
+    )
+    (fp_text value 1K (at 0 2.1) (layer F.Fab)
       (effects (font (size 1 1) (thickness 0.15)))
     )
@@
       (effects (font (size 1 1) (thickness 0.15)))
     )
-    (fp_text value 220R (at 2.54 0 180) (layer F.Fab)
+    (fp_text value 220R (at 0 2.1 180) (layer F.Fab)
       (effects (font (size 1 1) (thickness 0.15)))
     )
@@
     (tags "resistor 0805")
     (attr smd)
-    (fp_text reference R6 (at 0 -2.1 270) (layer F.SilkS) hide
-      (effects (font (size 1 1) (thickness 0.15)))
-    )
-    (fp_text value 10K (at -3.81 0 270) (layer F.Fab)
+    (fp_text reference R6 (at 0 -2.1 270) (layer F.SilkS)
+      (effects (font (size 1 1) (thickness 0.15)))
+    )
+    (fp_text value 10K (at 0 2.1 270) (layer F.Fab)
       (effects (font (size 1 1) (thickness 0.15)))
     )
@@
       (effects (font (size 1 1) (thickness 0.15)))
     )
-    (fp_text value ATTINY2313-P (at 3.81 11.43 90) (layer F.Fab)
+    (fp_text value ATTINY2313-P (at 3.81 25.25) (layer F.Fab)
       (effects (font (size 1 1) (thickness 0.15)))
     )
@@
     (tags "smd diode")
     (attr smd)
-    (fp_text reference D2 (at 0 1.6 270) (layer F.SilkS) hide
-      (effects (font (size 1 1) (thickness 0.15)))
-    )
-    (fp_text value D (at 0 -1.6 270) (layer F.Fab) hide
+    (fp_text reference D2 (at 0 1.6 270) (layer F.SilkS)
+      (effects (font (size 1 1) (thickness 0.15)))
+    )
+    (fp_text value D (at 0 -1.6 270) (layer F.Fab)
       (effects (font (size 1 1) (thickness 0.15)))
     )
@@
       (effects (font (size 1 1) (thickness 0.15)))
     )
-    (fp_text value D (at 0 -1.6 270) (layer F.Fab) hide
+    (fp_text value D (at 0 -1.6 270) (layer F.Fab)
       (effects (font (size 1 1) (thickness 0.15)))
     )
@@
     (tags "smd diode")
     (attr smd)
-    (fp_text reference D4 (at 0 1.6 270) (layer F.SilkS) hide
-      (effects (font (size 1 1) (thickness 0.15)))
-    )
-    (fp_text value D (at 0 -1.6 270) (layer F.Fab) hide
+    (fp_text reference D4 (at 0 1.6 270) (layer F.SilkS)
+      (effects (font (size 1 1) (thickness 0.15)))
+    )
+    (fp_text value D (at 0 -1.6 270) (layer F.Fab)
       (effects (font (size 1 1) (thickness 0.15)))
     )
@@
     (descr "SOT126, SOT32, Housing, Vertical,")
     (tags "SOT126, SOT32, Housing, Vertical,")
-    (fp_text reference Q2 (at 0.09906 -3.79984) (layer F.SilkS) hide
+    (fp_text reference Q2 (at 0.09906 -3.79984) (layer F.SilkS)
       (effects (font (size 1 1) (thickness 0.15)))
     )
@@
     (descr "Non Isolated JEDEC TO-220 Package")
     (tags "Power Integration YN Package")
-    (fp_text reference U1 (at 0 -4.318) (layer F.SilkS) hide
-      (effects (font (size 1 1) (thickness 0.15)))
-    )
-    (fp_text value LM7805CT (at 8.89 0) (layer F.Fab)
+    (fp_text reference U1 (at 0 -4.318) (layer F.SilkS)
+      (effects (font (size 1 1) (thickness 0.15)))
+    )
+    (fp_text value LM7805CT (at 0 -4.318) (layer F.Fab)
       (effects (font (size 1 1) (thickness 0.15)))
     )
@@
     (fp_line (start -1.55 -1.55) (end -1.55 1.55) (layer F.SilkS) (width 0.15))
     (fp_line (start -1.55 1.55) (end 0 1.55) (layer F.SilkS) (width 0.15))
-    (pad 1 thru_hole rect (at 0 0) (size 1.6 1.6) (drill 0.8) (layers *.Cu *.Mask)
+    (pad 1 thru_hole rect (at 0 0) (size 2.2352 2.2352) (drill 1.016) (layers *.Cu *.Mask)
       (net 4 "Net-(IC1-Pad1)"))
     (model Socket_Strips.3dshapes/Socket_Strip_Straight_1x01.wrl
@@
     (descr "Through hole socket strip")
     (tags "socket strip")
-    (fp_text reference P7 (at 0 -5.1 180) (layer F.SilkS) hide
-      (effects (font (size 1 1) (thickness 0.15)))
-    )
-    (fp_text value "+12V PWR" (at 0 -2.54 180) (layer F.Fab)
-      (effects (font (size 1 1) (thickness 0.15)))
-    )
+    (fp_text reference P7 (at 0 -5.1 180) (layer F.SilkS)
+      (effects (font (size 1 1) (thickness 0.15)))
+    )
+    (fp_text value "+12V PWR" (at 0 -3.1 180) (layer F.Fab)
+      (effects (font (size 1 1) (thickness 0.15)))
+    )
